Commit message: updated files

File: g_arm_description/urdf/robot_electromagnet.urdf.xacro (robot description, xacro)
@@ -1,4 +1,5 @@
 <?xml version="1.0"?>
-<robot name="g_arm">
+<robot name="g_arm" xmlns:xacro="http://www.ros.org/wiki/xacro">
+  <xacro:include filename="$(find g_arm_description)/urdf/g_arm_ros2_control.xacro"/>
   <!-- Definition of the base link -->
   <link name="base_link">

File: g_arm_moveit2/config/g_arm.ros2_control.xacro (robot description, xacro)
@@ -2,9 +2,12 @@
 <robot xmlns:xacro="http://www.ros.org/wiki/xacro">
     <xacro:macro name="g_arm_ros2_control" params="name initial_positions_file">
-        <xacro:property name="initial_positions" value="${load_yaml(initial_positions_file)['initial_positions']}"/>
+        <xacro:property name="initial_positions" value="${xacro.load_yaml(initial_positions_file)['initial_positions']}"/>
         <ros2_control name="${name}" type="system">
             <hardware>
                 <!-- By default, set up controllers for simulation. This won't work on real hardware -->
-                <plugin>mock_components/GenericSystem</plugin>
+                <plugin>mercer_g_arm_topic_hw/TopicSystem</plugin>
+                <param name="command_topic">/joint_commands</param>
+                <param name="feedback_topic">/joint_states_raw</param>
+                <!--plugin>mock_components/GenericSystem</plugin-->
             </hardware>
             <joint name="joint1">
@@ -13,5 +16,4 @@
                   <param name="initial_value">${initial_positions['joint1']}</param>
                 </state_interface>
-                <state_interface name="velocity"/>
             </joint>
             <joint name="joint2">
@@ -20,5 +22,4 @@
                   <param name="initial_value">${initial_positions['joint2']}</param>
                 </state_interface>
-                <state_interface name="velocity"/>
             </joint>
             <joint name="joint3">
@@ -27,5 +28,4 @@
                   <param name="initial_value">${initial_positions['joint3']}</param>
                 </state_interface>
-                <state_interface name="velocity"/>
             </joint>
             <joint name="jointPWM">
@@ -34,5 +34,4 @@
                   <param name="initial_value">${initial_positions['jointPWM']}</param>
                 </state_interface>
-                <state_interface name="velocity"/>
             </joint>
         </ros2_control>

File: g_arm_moveit2/config/g_arm.urdf.xacro (robot description, xacro)
@@ -5,5 +5,6 @@
     <xacro:include filename="$(find g_arm_description)/urdf/robot_electromagnet.urdf" />
     <!-- Import control_xacro -->
-    <xacro:include filename="g_arm.ros2_control.xacro" />
-    <xacro:g_arm_ros2_control name="FakeSystem" initial_positions_file="$(arg initial_positions_file)"/>
+    <xacro:include filename="$(find g_arm_moveit2)/config/g_arm.ros2_control.xacro" />
+    <!-- Include ros2_control configuration -->
+    <xacro:g_arm_ros2_control name="GArmTopicSystem" initial_positions_file="$(find g_arm_moveit2)/config/$(arg initial_positions_file)"/>
 </robot>

Commit message: Work from RPI

File: g_arm_description/urdf/robot_electromagnet.urdf.xacro (robot description, xacro)
@@ -411,5 +411,5 @@
     </collision>
   </link>
-  <joint name="jointPWM" type="revolute">
+  <joint name="jointPWM" type="fixed">
     <origin
       xyz="0.0 0.0 0.0"

File: g_arm_moveit2/config/g_arm.ros2_control.xacro (robot description, xacro)
@@ -8,5 +8,5 @@
                 <plugin>mercer_g_arm_topic_hw/TopicSystem</plugin>
                 <param name="command_topic">/joint_commands</param>
-                <param name="feedback_topic">/joint_states_raw</param>
+                <param name="feedback_topic">/joint_states</param>
                 <!--plugin>mock_components/GenericSystem</plugin-->
             </hardware>
