Commit message: Add TRAC_IK_SETUP.md, update robot_electromagnet.urdf

File: g_arm_description/urdf/robot_electromagnet.urdf (robot description, URDF)
Before this commit: robot g_arm, 15 links, 14 joints
Joints:
- joint joint1: limit lower=-1.5707 upper=1.5707 effort=200.0 velocity=200.0 -> lower=-1.7575 upper=1.7575 effort=200.0 velocity=200.0
