Commit message: removed remote bringup

File: ros2/src/g_arm_moveit2/config/g_arm.ros2_control.xacro (robot description, xacro)
@@ -1,13 +1,13 @@
 <?xml version="1.0"?>
 <robot xmlns:xacro="http://www.ros.org/wiki/xacro">
-    <xacro:macro name="g_arm_ros2_control" params="name initial_positions_file">
+    <xacro:macro name="g_arm_ros2_control" params="name initial_positions_file hardware_plugin:=mercer_g_arm_topic_hw/TopicSystem">
         <xacro:property name="initial_positions" value="${xacro.load_yaml(initial_positions_file)['initial_positions']}"/>
         <ros2_control name="${name}" type="system">
             <hardware>
-                <!-- By default, set up controllers for simulation. This won't work on real hardware -->
-                <plugin>mercer_g_arm_topic_hw/TopicSystem</plugin>
-                <param name="command_topic">/joint_commands</param>
-                <param name="feedback_topic">/joint_states</param>
-                <!--plugin>mock_components/GenericSystem</plugin-->
+                <plugin>${hardware_plugin}</plugin>
+                <xacro:if value="${hardware_plugin == 'mercer_g_arm_topic_hw/TopicSystem'}">
+                    <param name="command_topic">/joint_commands</param>
+                    <param name="feedback_topic">/joint_states</param>
+                </xacro:if>
             </hardware>
             <joint name="joint1">

File: ros2/src/g_arm_moveit2/config/g_arm.urdf.xacro (robot description, xacro)
@@ -2,4 +2,5 @@
 <robot xmlns:xacro="http://www.ros.org/wiki/xacro" name="g_arm">
     <xacro:arg name="initial_positions_file" default="initial_positions.yaml" />
+    <xacro:arg name="ros2_control_hardware_type" default="mercer_g_arm_topic_hw/TopicSystem" />
     <!-- Import g_arm urdf file -->
     <xacro:include filename="$(find g_arm_description)/urdf/robot_electromagnet.urdf" />
@@ -7,4 +8,4 @@
     <xacro:include filename="$(find g_arm_moveit2)/config/g_arm.ros2_control.xacro" />
     <!-- Include ros2_control configuration -->
-    <xacro:g_arm_ros2_control name="GArmTopicSystem" initial_positions_file="$(find g_arm_moveit2)/config/$(arg initial_positions_file)"/>
+    <xacro:g_arm_ros2_control name="GArmTopicSystem" initial_positions_file="$(find g_arm_moveit2)/config/$(arg initial_positions_file)" hardware_plugin="$(arg ros2_control_hardware_type)"/>
 </robot>
